File: PCB/QuickAccessBoard.kicad_pcb (KiCad board)
At the start: 2 copper layers, 90 x 81 mm, 27 parts, among them J1 OLED Display, SW1 SW_Push, SW10 SW_Push, SW11 SW_Push, SW12 SW_Push, SW13 RotaryEncoder_Switch, SW2 SW_Push, SW3 SW_Push, SW4 SW_Push, SW5 SW_Push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

Commit message: Fixed flaw in PCB
Routing:
- net C2: track 54.5 -> 73.7 mm, vias 0 -> 1
- net GND: track 62.0 -> 69.0 mm
Changed lines of the file:
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@@
+	)
+	(segment
+		(start 165.31276 38.57)
+		(end 164.225 38.57)
+		(width 0.2)
+		(layer "F.Cu")
+		(net 1)
 	)
 	(segment
@@
 	)
 	(segment
+		(start 167.376 40.63324)
+		(end 165.31276 38.57)
+		(width 0.2)
+		(layer "F.Cu")
+		(net 1)
+	)
+	(segment
 		(start 160.534 34.879)
 		(end 164.225 38.57)
+		(width 0.2)
+		(layer "F.Cu")
+		(net 1)
+	)
+	(segment
+		(start 169.1 42.9)
+		(end 167.376 41.176)
+		(width 0.2)
+		(layer "F.Cu")
+		(net 1)
+	)
+	(segment
+		(start 167.376 41.176)
+		(end 167.376 40.63324)
 		(width 0.2)
 		(layer "F.Cu")
@@
 	)
 	(segment
+		(start 158.01 95.11)
+		(end 169.86 95.11)
+		(width 0.2)
+		(layer "F.Cu")
+		(net 24)
+	)
+	(segment
+		(start 169.86 95.11)
+		(end 170 95.25)
+		(width 0.2)
+		(layer "F.Cu")
+		(net 24)
+	)
+	(segment
 		(start 177.17 56.98)
 		(end 177.17 95.07)
@@
 		(net 24)
 	)
+	(via
+		(at 170 95.25)
+		(size 0.6)
+		(drill 0.3)
+		(layers "F.Cu" "B.Cu")
+		(net 24)
+	)
 	(segment
 		(start 177.17 56.98)
@@
 		(width 0.2)
 		(layer "B.Cu")
+		(net 24)
+	)
+	(segment
+		(start 170 95.25)
+		(end 170.18 95.07)
+		(width 0.2)
+		(layer "B.Cu")
+		(net 24)
+	)
+	(segment
+		(start 170.18 95.07)
+		(end 177.17 95.07)
+		(width 0.2)
+		(layer "B.Cu")
